File: 2e0_pcb/2e0_pcb.kicad_pcb (KiCad board)
At the start: 2 copper layers, 100 x 100 mm, 53 parts, among them J1 Conn_01x02, J2 Conn_01x02, J3 Jack-DC, J4 Conn_01x02, J5 Conn_Coaxial, M1 Barrel_Polarity, M2 Logo_10mmx10mm, Q1 BC547CBU, SW1 SW_DPDT_x2, SW2 SW_DPDT_x2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

Commit message: Added changes from testing
Parts:
- C2, C4: value 12p -> 10p
- Q1, U1: footprint Package_TO_SOT_THT:TO-92_Inline -> Package_TO_SOT_THT:TO-92L
- R6: value 1k -> 3k9
- U2: value 74AC14 -> 74HC04
- Y1: value ABL-3.579545MHZ-B2 -> 3.58MHz
- moved D1 0.25 mm to (163.0, 118.8)
- moved D3 0.25 mm to (169.0, 118.8)
Routing:
- net Net-(Q1-Pad2): track 10.8 -> 12.5 mm
